Commit message: Fix ROS 2 / MoveIt2 errors and improve joint handling
- Resolved multiple ROS 2 and MoveIt2 errors and warnings
- Updated urdf_parser.py to collect joint upper and lower bounds
- Fixed issues with joints exceeding range limits
- Replaced joint position dictionary with parallel lists
  (separate joint names and positions)
- Integrated AUTOGLUON ensemble model

File: src/camera_system/urdf/camera_gazebo.xacro (robot description, xacro)
@@ -23,5 +23,5 @@
             <update_rate>30</update_rate>
             <camera>
-                <horizontal_fov>1.5708</horizontal_fov>
+                <horizontal_fov>1.3</horizontal_fov>
                 <image>
                     <width>640</width>

File: src/humanoid_robot/model/support/arm_3dof.xacro (robot description, xacro)
@@ -13,10 +13,10 @@
     <xacro:property name="twist_arm_length" value="${1-(revolute_arm_length*2)}"/>
     <link name="arm_base_link">
-        <!-- <visual>
+        <visual>
             <geometry>
                 <box size="${arm_base_length} ${arm_base_width} ${arm_base_height}"/>
             </geometry>
             <origin xyz="0.0 0.0 ${arm_base_height/2}" rpy="0.0 0.0 0.0"/>
-            <material name="orange"/>
+            <material name="black"/>
         </visual>
         <collision>
@@ -25,10 +25,10 @@
             </geometry>
             <origin xyz="0.0 0.0 ${arm_base_height/2}" rpy="0.0 0.0 0.0"/>
-        </collision> -->
+        </collision>
         <xacro:box_inertia m="0.5" l="${arm_base_length}" w="${arm_base_width}" h="${arm_base_height}"
                            xyz="0.0 0.0 ${arm_base_height/2.0}" rpy="0.0 0.0 0.0" />
     </link>
     <link name="link1">
-        <!-- <visual>
+        <visual>
             <geometry>
                 <cylinder radius="${arm_radius}" length="${link1_length}"/>
@@ -42,10 +42,10 @@
             </geometry>
             <origin xyz="0.0 0.0 ${link1_length/2}" rpy="0.0 0.0 0.0"/>
-        </collision> -->
+        </collision>
         <xacro:cylinder_inertia m="0.3" r="${arm_radius}" h="${link1_length}"
                                 xyz="0.0 0.0 ${link1_length/2}" rpy="0.0 0.0 0.0" />
     </link>
     <link name="link2">
-        <!-- <visual>
+        <visual>
             <geometry>
                 <cylinder radius="${arm_radius}" length="${revolute_arm_length}"/>
@@ -59,15 +59,15 @@
             </geometry>
             <origin xyz="0.0 0.0 ${revolute_arm_length/2}" rpy="0.0 0.0 0.0"/>
-        </collision> -->
+        </collision>
         <xacro:cylinder_inertia m="0.3" r="${arm_radius}" h="${revolute_arm_length}"
                                 xyz="0.0 0.0 ${revolute_arm_length/2}" rpy="0.0 0.0 0.0" />
     </link>
     <link name="link3">
-        <!-- <visual>
+        <visual>
             <geometry>
                 <cylinder radius="${arm_radius}" length="${revolute_arm_length}"/>
             </geometry>
             <origin xyz="0.0 0.0 ${revolute_arm_length/2}" rpy="0.0 0.0 0.0"/>
-            <material name="yellow"/>
+            <material name="red"/>
         </visual>
         <collision>
@@ -76,15 +76,15 @@
             </geometry>
             <origin xyz="0.0 0.0 ${revolute_arm_length/2}" rpy="0.0 0.0 0.0"/>
-        </collision> -->
+        </collision>
         <xacro:cylinder_inertia m="0.3" r="${arm_radius}" h="${revolute_arm_length}"
                                 xyz="0.0 0.0 ${revolute_arm_length/2}" rpy="0.0 0.0 0.0" />
     </link>
     <link name="link4">
-        <!-- <visual>
+        <visual>
             <geometry>
                 <cylinder radius="${arm_radius}" length="${twist_arm_length}"/>
             </geometry>
             <origin xyz="0.0 0.0 ${twist_arm_length/2}" rpy="0.0 0.0 0.0"/>
-            <material name="orange"/>
+            <material name="blue"/>
         </visual>
         <collision>
@@ -93,5 +93,5 @@
             </geometry>
             <origin xyz="0.0 0.0 ${twist_arm_length/2}" rpy="0.0 0.0 0.0"/>
-        </collision> -->
+        </collision>
         <xacro:cylinder_inertia m="0.3" r="${arm_radius}" h="${twist_arm_length}"
                                 xyz="0.0 0.0 ${twist_arm_length/2}" rpy="0.0 0.0 0.0" />
@@ -119,5 +119,5 @@
         <!-- <dynamics damping="1.0" friction="1.0"/> -->
     </joint>
-    <joint name="link3_link4_joint" type="continuous">
+    <joint name="link3_link4_joint" type="revolute">
         <parent link="link3"/>
         <child link="link4"/>

File: src/humanoid_robot/model/support/common_properties.xacro (robot description, xacro)
@@ -12,4 +12,10 @@
     <material name="yellow">
         <color rgba="1.0 1.0 0.0 1.0"/>
+    </material>
+    <material name="black">
+        <color rgba="0 0 0 1"/>
+    </material>
+    <material name="red">
+        <color rgba="1 0 0 1"/>
     </material>
     <xacro:macro name="box_inertia" params="m l w h xyz rpy">
